Commit message: Changed block grasp direction and corresponding urdf files

File: examples/pybullet/gym/pybullet_data/block_rot.urdf (robot description, URDF)
Before this commit: robot block_2, 1 links, 0 joints
Links:
- link block_2_base_link: geometry collision box size=0.1 0.005 0.005; visual box size=0.1 0.005 0.005
