Commit message: Centered torus obj file

File: examples/pybullet/gym/pybullet_data/torus/torus.urdf (robot description, URDF)
Before this commit: robot cube.urdf, 1 links, 0 joints
Links:
- link baseLink: geometry collision mesh filename=torus_only.obj scale=.01 .01 .01; visual mesh filename=torus_only.obj scale=.01 .01 .01
